File: PCB/CrystalSequencer.kicad_pcb (KiCad board)
At the start: 2 copper layers, 192.7 x 190 mm, 118 parts, among them J1 JACK_TRS_6PINS, J2 USB_C_Receptacle, J3 Conn_02x03_Odd_Even, SW1 SW_Push, SW10 SW_Push, SW11 SW_Push, SW12 SW_Push, SW13 SW_Push, SW14 SW_Push, SW15 SW_Push, SW16 SW_Push, SW17 SW_Push, SW2 SW_Push, SW3 SW_Push, SW4 SW_Push, SW5 SW_Push, SW6 SW_Push, SW7 SW_Push, SW8 SW_Push, SW9 SW_Push, U1 ATmega328P-A, U2 CD4051B, U3 OPA196xD, U4 ISD4004, U5 CH340C, X1 PAD0, X2 PAD1, X3 PAD2, X4 PAD3, X5 PAD4, X6 PAD5, X7 PAD6, X8 PAD7, Y1 16MHz

Commit message: Sent to PCB manuafcruting Yeah
Parts:
- added G***: LOGO, GaudiLabsLogos:MirnadaEnergyCommunity, B.Cu at (26.3, 69.3)
- added G***: LOGO, GaudiLabsLogos:CrystalHeartEmpty, B.Cu at (126.1, 78.4)
- added G***: LOGO, GaudiLabsLogos:CrystalHeartEmpty, B.Cu at (126.0, 94.0)
- added G***: LOGO, GaudiLabsLogos:GaudiLabs_8, B.Cu at (24.1, 59.4)
- added REF**: CrystalHolder, GaudiLabsFootPrints:CrystalHolder, F.Cu at (158.7, 35.7)
- added REF**: CrystalHolder, GaudiLabsFootPrints:CrystalHolder, F.Cu at (101.5, 30.8)
- added REF**: CrystalHolder, GaudiLabsFootPrints:CrystalHolder, F.Cu at (147.9, 146.3)
- added REF**: CrystalHolder, GaudiLabsFootPrints:CrystalHolder, F.Cu at (111.7, 169.9)
- added REF**: CrystalHolder, GaudiLabsFootPrints:CrystalHolder, F.Cu at (56.4, 57.5)
- added REF**: CrystalHolder, GaudiLabsFootPrints:CrystalHolder, F.Cu at (181.9, 76.3)
- added REF**: CrystalHolder, GaudiLabsFootPrints:CrystalHolder, F.Cu at (180.5, 117.4)
- added REF**: CrystalHolder, GaudiLabsFootPrints:CrystalHolder, F.Cu at (31.9, 87.1)
- moved G*** 76.4 mm to (17.8, 57.5), turned to -90 degrees
- moved G*** 59.6 mm to (123.1, 13.4), turned to -172 degrees
- moved G*** 52.8 mm to (67.6, 22.0), turned to -172 degrees
- moved G*** 45.9 mm to (17.8, 118.2), turned to -90 degrees
- moved G*** 44.2 mm to (182.3, 30.1), turned to 157.5 degrees
- moved G*** 37.2 mm to (144.6, 15.2), turned to 157.5 degrees
- moved G*** 28.8 mm to (38.7, 28.3), turned to -146.5 degrees
- moved G*** 20.4 mm to (105.4, 191.6), turned to -32.5 degrees
- moved SW16 19.7 mm to (108.4, 186.6), turned to -32.5 degrees
- moved H1 19.5 mm to (119.7, 186.8), turned to 26.5 degrees
- moved R13 19.4 mm to (100.6, 183.1), turned to 57.5 degrees
- moved G*** 19.2 mm to (76.0, 173.0), turned to -32.5 degrees
- moved H3 19.0 mm to (24.9, 132.5), turned to 26.5 degrees
- moved J1 18.9 mm to (46.9, 153.0), turned to 57.5 degrees
- moved G*** 18.8 mm to (135.2, 182.7), turned to 35 degrees
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Connections:
- SW1 pad 2: SW0 -> SW1
- SW10 pad 1: SW1 -> SW2
- SW11 pad 1: SW2 -> SW3
- SW12 pad 1: SW3 -> SW4
- SW13 pad 1: SW4 -> SW5
- SW14 pad 1: SW5 -> SW6
- SW15 pad 1: SW6 -> SW7
- SW16 pad 1: SW7 -> SW8
- SW17 pad 2: SW8 -> SW9
- SW2 pad 2: SW1 -> SW2
- SW3 pad 2: SW2 -> SW3
- SW4 pad 2: SW3 -> SW4
- SW5 pad 2: SW4 -> SW5
- SW6 pad 2: SW5 -> SW6
- SW7 pad 2: SW6 -> SW7
- SW8 pad 2: SW7 -> SW8
- SW9 pad 1: SW0 -> SW1
- U1 pad 11: SW8 -> SW9
- U2 pad 1: SW4 -> SW5
- U2 pad 12: SW3 -> SW4
- U2 pad 13: SW0 -> SW1
- U2 pad 14: SW1 -> SW2
- U2 pad 15: SW2 -> SW3
- U2 pad 2: SW6 -> SW7
- U2 pad 4: SW7 -> SW8
- U2 pad 5: SW5 -> SW6
- X1 pad 1: SW0 -> SW1
- X2 pad 1: SW1 -> SW2
- X3 pad 1: SW2 -> SW3
- X4 pad 1: SW3 -> SW4
- X5 pad 1: SW4 -> SW5
- X6 pad 1: SW5 -> SW6
- X7 pad 1: SW6 -> SW7
- X8 pad 1: SW7 -> SW8
Routing:
- net SW0: track 196.5 -> 0.00 mm, vias 2 -> 0
- net SW8: track 85.4 -> 210.4 mm, vias 2 -> 6
- net SW9: track 0.00 -> 85.4 mm, vias 0 -> 2
- net SW1: track 184.1 -> 241.4 mm, vias 2 -> 6
- net SW3: track 185.4 -> 235.1 mm
- net SW4: track 160.9 -> 209.1 mm, vias 2 -> 9
- net SW5: track 137.4 -> 175.7 mm, vias 3 -> 4
- net GND: track 67.9 -> 94.9 mm, vias 18 -> 20
- net SW7: track 177.5 -> 157.0 mm, vias 4 -> 7
- net Net-(D7-Pad1): track 153.3 -> 164.7 mm
- net SW2: track 205.9 -> 197.6 mm
- net VCC: track 1196.5 -> 1201.7 mm
- net SW6: track 152.9 -> 148.4 mm, vias 6 -> 5
- net Net-(D1-Pad1): track 61.3 -> 63.3 mm
- net Net-(R12-Pad1): track 16.6 -> 18.2 mm
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- added copper zone on F.Cu, net SW1
- added copper zone on F.Cu, net SW2
- added copper zone on F.Cu, net SW3
- added copper zone on F.Cu, net SW4
- added copper zone on F.Cu, net SW5
- added copper zone on F.Cu, net SW6
- added copper zone on F.Cu, net SW7
- added copper zone on F.Cu, net SW8
Other:
- board size 192.7 x 190 mm -> 185.7 x 188.8 mm
- board text added: "Make More Love"
- board text added: "X1"
- board text added: "X2"
- board text added: "X3"
- board text added: "X4"
- board text added: "X5"
- board text added: "X6"
- board text added: "X8"
- board text added: "gaudi.ch"
