File: PCB/CrystalSequencer.kicad_sch (KiCad schematic)
At the start: 92 parts, among them J1 JACK_TRS_6PINS, J2 USB_C_Receptacle, J3 Conn_02x03_Odd_Even, SW1 SW_Push, SW10 SW_Push, SW11 SW_Push, SW12 SW_Push, SW13 SW_Push, SW14 SW_Push, SW15 SW_Push, SW16 SW_Push, SW17 SW_Push, SW2 SW_Push, SW3 SW_Push, SW4 SW_Push, SW5 SW_Push, SW6 SW_Push, SW7 SW_Push, SW8 SW_Push, SW9 SW_Push, U1 ATmega328P-A, U2 CD4051B, U3 OPA196xD, U4 ISD4004, U5 CH340C, X1 PAD0, X2 PAD1, X3 PAD2, X4 PAD3, X5 PAD4, X6 PAD5, X7 PAD6, X8 PAD7, Y1 16MHz

Commit message: Sent to PCB manuafcruting Yeah
Connections:
- net SW0 is gone; now on net SW1: SW1.2, SW9.1, U2.13 (X0), X1.1
- net SW1: no longer SW10.1, SW2.2, U2.14 (X1), X2.1
- net SW2: now also SW10.1, SW2.2, U2.14 (X1), X2.1; no longer SW11.1, SW3.2, U2.15 (X2), X3.1
- net SW3: now also SW11.1, SW3.2, U2.15 (X2), X3.1; no longer SW12.1, SW4.2, U2.12 (X3), X4.1
- net SW4: now also SW12.1, SW4.2, U2.12 (X3), X4.1; no longer SW13.1, SW5.2, U2.1 (X4), X5.1
- net SW5: now also SW13.1, SW5.2, U2.1 (X4), X5.1; no longer SW14.1, SW6.2, U2.5 (X5), X6.1
- net SW6: now also SW14.1, SW6.2, U2.5 (X5), X6.1; no longer SW15.1, SW7.2, U2.2 (X6), X7.1
- net SW7: now also SW15.1, SW7.2, U2.2 (X6), X7.1; no longer SW16.1, SW8.2, U2.4 (X7), X8.1
- net SW8: now also SW16.1, SW8.2, U2.4 (X7), X8.1; no longer SW17.2, U1.11 (PD7)
- new net SW9: SW17.2, U1.11 (PD7)
Changed lines of the file:
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@@
     )
   )
-  (global_label "SW0" (shape input) (at 187.96 158.75 180) (fields_autoplaced)
-    (effects (font (size 1.27 1.27)) (justify right))
-    (property "Intersheet References" "${INTERSHEET_REFS}" (id 0) (at 181.6764 158.8294 0)
+  (global_label "SW1" (shape input) (at 187.96 158.75 180) (fields_autoplaced)
+    (effects (font (size 1.27 1.27)) (justify right))
+    (property "Intersheet References" "${INTERSHEET_REFS}" (id 0) (at 181.6764 158.6706 0)
       (effects (font (size 1.27 1.27)) (justify right) hide)
     )
@@
     )
   )
-  (global_label "SW2" (shape input) (at 188.595 172.72 180) (fields_autoplaced)
-    (effects (font (size 1.27 1.27)) (justify right))
-    (property "Intersheet References" "${INTERSHEET_REFS}" (id 0) (at 182.3114 172.7994 0)
+  (global_label "SW3" (shape input) (at 188.595 172.72 180) (fields_autoplaced)
+    (effects (font (size 1.27 1.27)) (justify right))
+    (property "Intersheet References" "${INTERSHEET_REFS}" (id 0) (at 182.3114 172.6406 0)
       (effects (font (size 1.27 1.27)) (justify right) hide)
     )
@@
     )
   )
-  (global_label "SW1" (shape input) (at 187.96 165.735 180) (fields_autoplaced)
-    (effects (font (size 1.27 1.27)) (justify right))
-    (property "Intersheet References" "${INTERSHEET_REFS}" (id 0) (at 181.6764 165.8144 0)
-      (effects (font (size 1.27 1.27)) (justify right) hide)
-    )
-  )
-  (global_label "SW8" (shape input) (at 89.535 215.265 0) (fields_autoplaced)
-    (effects (font (size 1.27 1.27)) (justify left))
-    (property "Intersheet References" "${INTERSHEET_REFS}" (id 0) (at 95.8186 215.3444 0)
-      (effects (font (size 1.27 1.27)) (justify left) hide)
-    )
-  )
-  (global_label "SW0" (shape input) (at 50.8 59.69 180) (fields_autoplaced)
-    (effects (font (size 1.27 1.27)) (justify right))
-    (property "Intersheet References" "${INTERSHEET_REFS}" (id 0) (at 44.5164 59.7694 0)
+  (global_label "SW2" (shape input) (at 187.96 165.735 180) (fields_autoplaced)
+    (effects (font (size 1.27 1.27)) (justify right))
+    (property "Intersheet References" "${INTERSHEET_REFS}" (id 0) (at 181.6764 165.6556 0)
+      (effects (font (size 1.27 1.27)) (justify right) hide)
+    )
+  )
+  (global_label "SW9" (shape input) (at 89.535 215.265 0) (fields_autoplaced)
+    (effects (font (size 1.27 1.27)) (justify left))
+    (property "Intersheet References" "${INTERSHEET_REFS}" (id 0) (at 95.8186 215.1856 0)
+      (effects (font (size 1.27 1.27)) (justify left) hide)
+    )
+  )
+  (global_label "SW1" (shape input) (at 50.8 59.69 180) (fields_autoplaced)
+    (effects (font (size 1.27 1.27)) (justify right))
+    (property "Intersheet References" "${INTERSHEET_REFS}" (id 0) (at 44.5164 59.6106 0)
       (effects (font (size 1.27 1.27)) (justify right) hide)
     )
@@
     )
   )
-  (global_label "SW3" (shape input) (at 50.8 76.835 180) (fields_autoplaced)
+  (global_label "SW4" (shape input) (at 50.8 76.835 180) (fields_autoplaced)
     (effects (font (size 1.27 1.27)) (justify right))
     (property "Intersheet References" "${INTERSHEET_REFS}" (id 0) (at 44.5164 76.7556 0)
@@
     )
   )
-  (global_label "SW6" (shape input) (at 188.595 200.66 180) (fields_autoplaced)
-    (effects (font (size 1.27 1.27)) (justify right))
-    (property "Intersheet References" "${INTERSHEET_REFS}" (id 0) (at 182.3114 200.7394 0)
+  (global_label "SW7" (shape input) (at 188.595 200.66 180) (fields_autoplaced)
+    (effects (font (size 1.27 1.27)) (justify right))
+    (property "Intersheet References" "${INTERSHEET_REFS}" (id 0) (at 182.3114 200.5806 0)
       (effects (font (size 1.27 1.27)) (justify right) hide)
     )
@@
     )
   )
-  (global_label "SW8" (shape input) (at 203.2 219.075 180) (fields_autoplaced)
+  (global_label "SW9" (shape input) (at 203.2 219.075 180) (fields_autoplaced)
     (effects (font (size 1.27 1.27)) (justify right))
     (property "Intersheet References" "${INTERSHEET_REFS}" (id 0) (at 196.9164 218.9956 0)
@@
     )
   )
-  (global_label "SW3" (shape input) (at 188.595 179.07 180) (fields_autoplaced)
-    (effects (font (size 1.27 1.27)) (justify right))
-    (property "Intersheet References" "${INTERSHEET_REFS}" (id 0) (at 182.3114 179.1494 0)
+  (global_label "SW4" (shape input) (at 188.595 179.07 180) (fields_autoplaced)
+    (effects (font (size 1.27 1.27)) (justify right))
+    (property "Intersheet References" "${INTERSHEET_REFS}" (id 0) (at 182.3114 178.9906 0)
       (effects (font (size 1.27 1.27)) (justify right) hide)
     )
@@
     )
   )
-  (global_label "SW4" (shape input) (at 188.595 186.055 180) (fields_autoplaced)
-    (effects (font (size 1.27 1.27)) (justify right))
-    (property "Intersheet References" "${INTERSHEET_REFS}" (id 0) (at 182.3114 186.1344 0)
+  (global_label "SW5" (shape input) (at 188.595 186.055 180) (fields_autoplaced)
+    (effects (font (size 1.27 1.27)) (justify right))
+    (property "Intersheet References" "${INTERSHEET_REFS}" (id 0) (at 182.3114 185.9756 0)
       (effects (font (size 1.27 1.27)) (justify right) hide)
     )
@@
     )
   )
-  (global_label "SW4" (shape input) (at 50.8 82.55 180) (fields_autoplaced)
+  (global_label "SW5" (shape input) (at 50.8 82.55 180) (fields_autoplaced)
     (effects (font (size 1.27 1.27)) (justify right))
     (property "Intersheet References" "${INTERSHEET_REFS}" (id 0) (at 44.5164 82.4706 0)
@@
     )
   )
-  (global_label "SW2" (shape input) (at 50.8 71.12 180) (fields_autoplaced)
+  (global_label "SW3" (shape input) (at 50.8 71.12 180) (fields_autoplaced)
     (effects (font (size 1.27 1.27)) (justify right))
     (property "Intersheet References" "${INTERSHEET_REFS}" (id 0) (at 44.5164 71.0406 0)
@@
     )
   )
-  (global_label "SW5" (shape input) (at 188.595 193.675 180) (fields_autoplaced)
-    (effects (font (size 1.27 1.27)) (justify right))
-    (property "Intersheet References" "${INTERSHEET_REFS}" (id 0) (at 182.3114 193.7544 0)
+  (global_label "SW6" (shape input) (at 188.595 193.675 180) (fields_autoplaced)
+    (effects (font (size 1.27 1.27)) (justify right))
+    (property "Intersheet References" "${INTERSHEET_REFS}" (id 0) (at 182.3114 193.5956 0)
       (effects (font (size 1.27 1.27)) (justify right) hide)
     )
@@
     )
   )
-  (global_label "SW7" (shape input) (at 188.595 207.645 180) (fields_autoplaced)
-    (effects (font (size 1.27 1.27)) (justify right))
-    (property "Intersheet References" "${INTERSHEET_REFS}" (id 0) (at 182.3114 207.7244 0)
+  (global_label "SW8" (shape input) (at 188.595 207.645 180) (fields_autoplaced)
+    (effects (font (size 1.27 1.27)) (justify right))
+    (property "Intersheet References" "${INTERSHEET_REFS}" (id 0) (at 182.3114 207.5656 0)
       (effects (font (size 1.27 1.27)) (justify right) hide)
     )
@@
     )
   )
-  (global_label "SW1" (shape input) (at 50.8 65.405 180) (fields_autoplaced)
+  (global_label "SW2" (shape input) (at 50.8 65.405 180) (fields_autoplaced)
     (effects (font (size 1.27 1.27)) (justify right))
     (property "Intersheet References" "${INTERSHEET_REFS}" (id 0) (at 44.5164 65.3256 0)
@@
     )
   )
-  (global_label "SW5" (shape input) (at 50.8 88.265 180) (fields_autoplaced)
+  (global_label "SW6" (shape input) (at 50.8 88.265 180) (fields_autoplaced)
     (effects (font (size 1.27 1.27)) (justify right))
     (property "Intersheet References" "${INTERSHEET_REFS}" (id 0) (at 44.5164 88.1856 0)
@@
     )
   )
-  (global_label "SW6" (shape input) (at 50.8 93.98 180) (fields_autoplaced)
+  (global_label "SW7" (shape input) (at 50.8 93.98 180) (fields_autoplaced)
     (effects (font (size 1.27 1.27)) (justify right))
     (property "Intersheet References" "${INTERSHEET_REFS}" (id 0) (at 44.5164 93.9006 0)
@@
     )
   )
-  (global_label "SW7" (shape input) (at 50.8 99.695 180) (fields_autoplaced)
+  (global_label "SW8" (shape input) (at 50.8 99.695 180) (fields_autoplaced)
     (effects (font (size 1.27 1.27)) (justify right))
     (property "Intersheet References" "${INTERSHEET_REFS}" (id 0) (at 44.5164 99.6156 0)
